File: digital lockin.brd (EAGLE design)
At the start: 76.2 x 94.9 mm, 24 parts, among them IC1 OPA2650E, IC2 LM358D, T2 NPN, U2 RASPBERRY_PICOSMD-TH, U5 TL431AIDBZR

Commit message: Eagle assignment 3 Jechiel van Dijk
Parts:
- moved C9 31.5 mm to (52.3, 49.8)
- moved C8 25.1 mm to (32.5, 14.2)
- moved C10 23.9 mm to (28.4, 5.08)
- moved C1 22.3 mm to (26.2, 11.7)
- moved PD1 20.5 mm to (26.7, 22.6)
- moved IC1 19.1 mm to (39.9, 12.7), turned to 0 degrees
- moved R6 13.7 mm to (43.9, 21.8)
- moved R8 13.0 mm to (12.2, 62.0)
- moved R3 11.7 mm to (42.2, 27.2), turned to 180 degrees
- moved U2 11.1 mm to (41.1, 80.0), turned to 270 degrees
- moved R9 8.27 mm to (68.8, 20.8), turned to 90 degrees
- moved T2 7.64 mm to (12.2, 17.3), turned to 0 degrees
- moved C3 6.51 mm to (55.6, 10.2)
- moved R1 6.12 mm to (17.8, 56.4)
- moved C2 5.40 mm to (61.2, 2.29)
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Connections:
- removed net SWGND: U2.42, U2.P$42
- removed net V+: IC1.8
- removed net V-: IC1.4
- new net N$1: C3.1, IC1.7, R6.2
- new net N$11: C1.1, IC1.2, PD1.K, R3.2, R6.1
- new net N$2: C3.2, IC1.6, R7.2
- new net N$5: C2.1, IC1.5, R5.2
- net 5V: now also C8.1, IC1.8
- net ADCMID: now also C2.2, R7.1, R9.2
- net AMPOUT: now also C1.2, IC1.1, R3.1, R5.1
- net GND: now also C10.1, C10.2, C8.2, IC1.3, IC1.4, PD1.A, R9.1, U2.42, U2.P$42
Routing:
- net 5V: track 0.00 -> 146.8 mm, vias 0 -> 5
- net ADCMID: track 0.00 -> 129.5 mm, vias 0 -> 2
- net AMPOUT: track 0.00 -> 88.5 mm, vias 0 -> 4
- net LEDCTRL: track 0.00 -> 80.4 mm
- net ADCREF: track 0.00 -> 63.0 mm
- net N$11: track 0.00 -> 59.1 mm
- net 3V3: track 0.00 -> 52.1 mm
- net N$5: track 0.00 -> 42.0 mm, vias 0 -> 2
- net N$2: track 0.00 -> 34.2 mm
- net N$9: track 0.00 -> 31.9 mm
- net N$1: track 0.00 -> 23.7 mm
- net N$10: track 0.00 -> 19.8 mm
- net N$20: track 0.00 -> 12.0 mm
- net N$3: track 0.00 -> 9.34 mm
- net GND: track 0.00 -> 7.97 mm, vias 4 -> 6
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- added copper zone on layer 1, net GND
- added copper zone on layer 16, net GND
